File: kicad/kicad.kicad_pcb (KiCad board)
At the start: 2 copper layers, 10 parts, among them M1 TP4056Module, U1 LT1963

Commit message: WIP
Parts:
- added C4: 0.01u, Capacitor_SMD:C_1206_3216Metric, F.Cu at (61.6, 105.7)
- added C5: 470u, Capacitor_THT:CP_Radial_D5.0mm_P2.50mm, F.Cu at (59.9, 111.2)
- added J1: Prog Pads, Connector_PinHeader_2.54mm:PinHeader_1x05_P2.54mm_Vertical, F.Cu at (53.1, 79.8)
- added J2: SLP, Connector_PinHeader_2.54mm:PinHeader_1x02_P2.54mm_Vertical, F.Cu at (53.6, 101.7)
- added J3: SHT21, Connector_PinSocket_2.54mm:PinSocket_1x04_P2.54mm_Vertical, F.Cu at (106.7, 95.7)
- added J4: BH1750, Connector_PinSocket_2.54mm:PinSocket_1x05_P2.54mm_Vertical, F.Cu at (102.1, 95.7)
- added R10: 470, Resistor_SMD:R_1206_3216Metric, F.Cu at (84.8, 99.3)
- added R5: 10k, Resistor_SMD:R_1206_3216Metric, F.Cu at (78.2, 74.4)
- added R6: 10k, Resistor_SMD:R_1206_3216Metric, F.Cu at (84.0, 74.6)
- added R7: 10k, Resistor_SMD:R_1206_3216Metric, F.Cu at (90.1, 74.5)
- added R8: 10k, Resistor_SMD:R_1206_3216Metric, F.Cu at (80.0, 99.3)
- added R9: 470, Resistor_SMD:R_1206_3216Metric, F.Cu at (90.2, 99.2)
- added SW1: RST, Button_Switch_SMD:SW_Push_SPST_NO_Alps_SKRK, F.Cu at (84.2, 93.4)
- added SW2: PRG, Button_Switch_SMD:SW_Push_SPST_NO_Alps_SKRK, F.Cu at (90.2, 93.3)
- added U2: ESP-12F, RF_Module:ESP-12E, F.Cu at (67.5, 90.2)
- R3: value R -> 1M
- R4: value R -> 220k
- moved M1 52.3 mm to (74.0, 33.0), turned to 270 degrees
- moved BT1 31.7 mm to (36.0, 34.0)
- moved R2 27.7 mm to (83.5, 55.1), turned to 90 degrees
- moved C1 25.1 mm to (78.3, 63.4), turned to 90 degrees
- moved R4 24.9 mm to (68.8, 71.3), turned to 0 degrees
- moved R1 23.4 mm to (83.3, 61.4), turned to 90 degrees
- moved U1 23.4 mm to (72.6, 59.6)
- moved C2 18.9 mm to (66.8, 55.1)
- moved R3 13.9 mm to (61.9, 71.5), turned to 0 degrees
- moved C3 13.4 mm to (90.2, 67.0), turned to 90 degrees
Connections:
- net Net-(C1-Pad1) renamed PWR
- net Net-(C2-Pad2) renamed GND
