File: pcb_charger/kicad.sch (KiCad schematic (older format))
At the start: 6 parts, among them J1 B+, J2 B-, J3 OUT+, J4 OUT-, M1 TP4056Module, SW1 SW_SPDT

Commit message: Last changes to the charger board and gerbers
Connections:
- net B+: now reaches J1.1 (Pin_1), M1.3 (B+)
- net B-: now reaches J2.1 (Pin_1), M1.4 (B-)
- net OUT+: now reaches M1.5 (OUT+), SW1.2 (B)
- net OUT-: now reaches J4.1 (Pin_1), M1.6 (OUT-)
- net OUT+on: now reaches J3.1 (Pin_1), SW1.1 (A)
Changed lines of the file:
@@
 	2800 1800 3100 1800
 NoConn ~ 2800 2000
+Text Label 1550 2400 0    50   ~ 0
+B+
+Text Label 1800 2400 0    50   ~ 0
+B-
+Text Label 2850 1800 0    50   ~ 0
+OUT+on
+Text Label 2350 2100 0    50   ~ 0
+OUT-
+Text Label 2300 1900 0    50   ~ 0
+OUT+
 $EndSCHEMATC
