File: pcb_esp/kicad.sch (KiCad schematic (older format))
At the start: 24 parts, among them J1 Prog Pads, J2 SLP, J3 SHT21, J4 BH1750, J5 PWRIN, J6 GND, SW1 RST, SW2 PRG, U1 LT1963, U2 ESP-12F

Commit message: Organise files a bit
Parts:
- C4: value 0.01u -> 100n
- R1: value 1M -> 750k
- R2: value 680k -> 510k
- R3: value 1M -> 3M3
- R4: value 220k -> 750k
Changed lines of the file:
@@
 P 5700 1050
 F 0 "R1" H 5770 1096 50  0000 L CNN
-F 1 "1M" H 5770 1005 50  0000 L CNN
+F 1 "750k" H 5770 1005 50  0000 L CNN
 F 2 "Resistor_SMD:R_1206_3216Metric" V 5630 1050 50  0001 C CNN
 F 3 "~" H 5700 1050 50  0001 C CNN
@@
 P 5700 1400
 F 0 "R2" H 5770 1446 50  0000 L CNN
-F 1 "680k" H 5770 1355 50  0000 L CNN
+F 1 "510k" H 5770 1355 50  0000 L CNN
 F 2 "Resistor_SMD:R_1206_3216Metric" V 5630 1400 50  0001 C CNN
 F 3 "~" H 5700 1400 50  0001 C CNN
@@
 P 3650 1050
 F 0 "R3" H 3720 1096 50  0000 L CNN
-F 1 "1M" H 3720 1005 50  0000 L CNN
+F 1 "3M3" H 3720 1005 50  0000 L CNN
 F 2 "Resistor_SMD:R_1206_3216Metric" V 3580 1050 50  0001 C CNN
 F 3 "~" H 3650 1050 50  0001 C CNN
@@
 P 3650 1400
 F 0 "R4" H 3720 1446 50  0000 L CNN
-F 1 "220k" H 3720 1355 50  0000 L CNN
+F 1 "750k" H 3720 1355 50  0000 L CNN
 F 2 "Resistor_SMD:R_1206_3216Metric" V 3580 1400 50  0001 C CNN
 F 3 "~" H 3650 1400 50  0001 C CNN
@@
 P 1500 3350
 F 0 "C4" H 1615 3396 50  0000 L CNN
-F 1 "0.01u" H 1615 3305 50  0000 L CNN
+F 1 "100n" H 1615 3305 50  0000 L CNN
 F 2 "Capacitor_SMD:C_1206_3216Metric_Pad1.42x1.75mm_HandSolder" H 1538 3200 50  0001 C CNN
 F 3 "~" H 1500 3350 50  0001 C CNN
